Commit message: first domus food scoop video

File: niryo_one_description/urdf/v2/niryo_one.urdf (robot description, URDF)
Before this commit: robot niryo_one, 9 links, 8 joints
Links:
- added link spoon_link
Joints:
- added joint hand_spoon_joint: type fixed, parent hand_link, child spoon_link, origin xyz=0.114 0.0 0.031 rpy=0 0 0

File: niryo_one_description/urdf/v2/niryo_one.urdf.xacro (robot description, xacro)
@@ -30,4 +30,8 @@
     <!-- not yet implemented, for now -->
     <xacro:property name="distance_hand_gripper" value="0.00" />
+    <!-- TSR 2018-19-07 Adding info about test spoon-->
+    <xacro:property name="spoon_offset_left" value="0.114" />
+    <xacro:property name="spoon_offset_up" value="0.0" />
+    <xacro:property name="spoon_offset_forward" value="0.031" />
 	<xacro:property name="thickness_arm_axis" value="0.052" />
 	<xacro:property name="thickness_forearm_axis" value="0.048" />
@@ -169,4 +173,6 @@
     <link name="gripper_link">
 	</link>
+    <link name="spoon_link">
+	</link>
 	<!--Joints -->
     <joint name="ground_joint" type="fixed">
@@ -221,4 +227,9 @@
         <child link="gripper_link" />
         <origin xyz="0 0 ${distance_hand_gripper}" rpy="${-PI/2} ${-PI/2} 0" />
+    </joint>
+	<joint name="hand_spoon_joint" type="fixed">
+        <parent link="hand_link" />
+        <child link="spoon_link" />
+        <origin xyz="${spoon_offset_left} ${spoon_offset_up} ${spoon_offset_forward}" rpy="0 0 0" />
 	</joint>
 </robot>

Commit message: lengthen spoon

File: niryo_one_description/urdf/v2/niryo_one.urdf (robot description, URDF)
Before this commit: robot niryo_one, 10 links, 9 joints
Joints:
- joint hand_spoon_joint: origin xyz=0.114 0.0 0.031 rpy=0 0 0 -> xyz=0.14 0.0 0.031 rpy=0 0 0

Commit message: not sure how adding these files breaks everything, but let's see

File: niryo_one_description/urdf/v2/niryo_one.urdf (robot description, URDF)
Before this commit: robot niryo_one, 10 links, 9 joints
Links:
- added link camera_rgb_optical_frame
Joints:
- added joint kinect_camera_joint: type fixed, parent base_link, child camera_rgb_optical_frame, origin xyz=0 -0.2 0 rpy=0 0 0
- joint hand_spoon_joint: origin xyz=0.14 0.0 0.031 rpy=0 0 0 -> xyz=0.114 0.0 0.031 rpy=0 0 0

File: niryo_one_description/urdf/v2/niryo_one.urdf.xacro (robot description, xacro)
@@ -175,4 +175,6 @@
     <link name="spoon_link">
 	</link>
+    <link name="camera_rgb_optical_frame">
+	</link>
 	<!--Joints -->
     <joint name="ground_joint" type="fixed">
@@ -233,3 +235,8 @@
         <origin xyz="${spoon_offset_left} ${spoon_offset_up} ${spoon_offset_forward}" rpy="0 0 0" />
 	</joint>
+    <joint name="kinect_camera_joint" type="fixed">
+        <parent link="base_link" />
+        <child link="camera_rgb_optical_frame" />
+        <origin xyz="0 -0.2 0" rpy="0 0 0" />
+	</joint>
 </robot>

Commit message: update spoon length to 14cm

File: niryo_one_description/urdf/v2/niryo_one.urdf (robot description, URDF)
Before this commit: robot niryo_one, 11 links, 10 joints
Joints:
- joint hand_spoon_joint: origin xyz=0.114 0.0 0.031 rpy=0 0 0 -> xyz=0.14 0.0 0.031 rpy=0 0 0

File: niryo_one_description/urdf/v2/niryo_one.urdf.xacro (robot description, xacro)
@@ -31,5 +31,5 @@
     <xacro:property name="distance_hand_gripper" value="0.00" />
     <!-- TSR 2018-19-07 Adding info about test spoon-->
-    <xacro:property name="spoon_offset_left" value="0.114" />
+    <xacro:property name="spoon_offset_left" value="0.14" />
     <xacro:property name="spoon_offset_up" value="0.0" />
     <xacro:property name="spoon_offset_forward" value="0.031" />

Commit message: demoed for myself and ate way more roasted salted corn than is probably healthy

File: niryo_one_description/urdf/v2/niryo_one.urdf (robot description, URDF)
Before this commit: robot niryo_one, 11 links, 10 joints
Joints:
- joint hand_spoon_joint: origin xyz=0.14 0.0 0.031 rpy=0 0 0 -> xyz=0.125 0.0 0.031 rpy=0 0 0

File: niryo_one_description/urdf/v2/niryo_one.urdf.xacro (robot description, xacro)
@@ -31,5 +31,5 @@
     <xacro:property name="distance_hand_gripper" value="0.00" />
     <!-- TSR 2018-19-07 Adding info about test spoon-->
-    <xacro:property name="spoon_offset_left" value="0.14" />
+    <xacro:property name="spoon_offset_left" value="0.125" />
     <xacro:property name="spoon_offset_up" value="0.0" />
     <xacro:property name="spoon_offset_forward" value="0.031" />
