Commit message: add spoon link and camera optical frame

File: niryo_one_description/urdf/v2/niryo_one.urdf.xacro (robot description, xacro)
@@ -21,10 +21,16 @@
     <xacro:property name="distance_arm_elbow_x" value="0.210" />
     <xacro:property name="distance_arm_elbow_y" value="0.0" />
-    <xacro:property name="distance_elbow_forearm_x" value="0.0415" />
-    <xacro:property name="distance_elbow_forearm_y" value="0.030" />
+    <xacro:property name="distance_elbow_forearm_x" value="0.037" />
+    <xacro:property name="distance_elbow_forearm_y" value="0.032" />
     <xacro:property name="distance_forearm_wrist_z" value="0.180" />
     <xacro:property name="distance_wrist_hand_x" value="0.0164" />
     <xacro:property name="distance_wrist_hand_y" value="-0.0055" />
     <xacro:property name="distance_hand_tool" value="0.0073" />
+    <!-- TSR 2018-19-07 Adding info about test spoon-->
+    <xacro:property name="spoon_offset_left" value="0.125" />
+    <xacro:property name="spoon_offset_up" value="0.0" />
+    <xacro:property name="spoon_offset_forward" value="0.031" />
+    <xacro:property name="thickness_arm_axis" value="0.052" />
+    <xacro:property name="thickness_forearm_axis" value="0.048" />
 	<xacro:property name="PI" value="3.14159265359" />
     <xacro:property name="limit_low_shoulder_rotation" value="-3.05433" />
@@ -142,4 +148,8 @@
     <link name="tool_link">
 	</link>
+    <link name="spoon_link">
+	</link>
+    <link name="camera_rgb_optical_frame">
+	</link>
 	<!--Joints -->
     <joint name="ground_joint" type="fixed">
@@ -194,4 +204,14 @@
         <child link="tool_link" />
         <origin xyz="0 0 ${distance_hand_tool}" rpy="${-PI/2} ${-PI/2} 0" />
+    </joint>
+	<joint name="hand_spoon_joint" type="fixed">
+        <parent link="hand_link" />
+        <child link="spoon_link" />
+        <origin xyz="${spoon_offset_left} ${spoon_offset_up} ${spoon_offset_forward}" rpy="0 0 0" />
+	</joint>
+    <joint name="kinect_camera_joint" type="fixed">
+        <parent link="base_link" />
+        <child link="camera_rgb_optical_frame" />
+        <origin xyz="0 -0.2 0" rpy="0 0 0" />
 	</joint>
 </robot>

Commit message: this runs fine, but is probably only partially solved. The plan is to _only_ change the name for the custom niryo robot

File: niryo_one_description/urdf/v2/niryo_one.urdf.xacro (robot description, xacro)
@@ -16,4 +16,6 @@
 -->
 <robot xmlns:xacro="http://www.ros.org/wiki/xacro" name="niryo_one">
+        <!-- Add an xacro arg to simulate tf_prefix -->
+    <xacro:arg name="link_prefix" default=""/>
 	<!-- Properties -->
     <xacro:property name="distance_origin_shoulder_z" value="0.103" />
@@ -47,6 +49,6 @@
     <xacro:property name="limit_up_hand_rotation" value="2.57436" />
 	<!-- Links -->
-    <link name="ground_link"/>
-    <link name="base_link">
+    <link name="$(arg link_prefix)ground_link"/>
+    <link name="$(arg link_prefix)base_link">
 		<visual>
 			<origin xyz="0 0 0" rpy="0 0 0" />
@@ -62,5 +64,5 @@
         </collision>
 	</link>
-    <link name="shoulder_link">
+    <link name="$(arg link_prefix)shoulder_link">
 		<visual>
 			<origin xyz="0 0 0" rpy="0 0 0" />
@@ -76,5 +78,5 @@
         </collision>
 	</link>
-    <link name="arm_link">
+    <link name="$(arg link_prefix)arm_link">
 		<visual>
 			<origin xyz="0 0 0" rpy="0 0 0" />
@@ -90,5 +92,5 @@
         </collision>
 	</link>
-    <link name="elbow_link">
+    <link name="$(arg link_prefix)elbow_link">
 		<visual>
 			<origin xyz="0 0 0" rpy="0 0 0" />
@@ -104,5 +106,5 @@
         </collision>
 	</link>
-    <link name="forearm_link">
+    <link name="$(arg link_prefix)forearm_link">
 		<visual>
 			<origin xyz="0 0 0" rpy="0 0 0" />
@@ -118,5 +120,5 @@
         </collision>
 	</link>
-    <link name="wrist_link">
+    <link name="$(arg link_prefix)wrist_link">
 		<visual>
 			<origin xyz="0 0 0" rpy="0 0 0" />
@@ -132,5 +134,5 @@
         </collision>
 	</link>
-    <link name="hand_link">
+    <link name="$(arg link_prefix)hand_link">
 		<visual>
 			<origin xyz="0 0 0" rpy="0 0 0" />
@@ -146,19 +148,19 @@
         </collision>
 	</link>
-    <link name="tool_link">
-	</link>
-    <link name="spoon_link">
-	</link>
-    <link name="camera_rgb_optical_frame">
+    <link name="$(arg link_prefix)tool_link">
+	</link>
+    <link name="$(arg link_prefix)spoon_link">
+	</link>
+    <link name="$(arg link_prefix)camera_rgb_optical_frame">
 	</link>
 	<!--Joints -->
     <joint name="ground_joint" type="fixed">
-        <parent link="ground_link" />
-        <child link="base_link" />
+        <parent link="$(arg link_prefix)ground_link" />
+        <child link="$(arg link_prefix)base_link" />
         <origin xyz="0 0 0" rpy="0 0 0" />
     </joint>
 	<joint name="joint_1" type="revolute">
-        <parent link="base_link" />
-        <child link="shoulder_link" />
+        <parent link="$(arg link_prefix)base_link" />
+        <child link="$(arg link_prefix)shoulder_link" />
 		<origin xyz="0 0 ${distance_origin_shoulder_z}" rpy="0 0 0" />
 		<axis xyz="0 0 1" />
@@ -166,6 +168,6 @@
 	</joint>
 	<joint name="joint_2" type="revolute">
-        <parent link="shoulder_link" />
-        <child link="arm_link" />
+        <parent link="$(arg link_prefix)shoulder_link" />
+        <child link="$(arg link_prefix)arm_link" />
         <origin xyz="0 0 ${distance_shoulder_arm_z}" rpy="${PI/2} ${-PI/2} 0" />
 		<limit effort="1" velocity="1.0" lower="${limit_low_arm_rotation}" upper="${limit_up_arm_rotation}" />
@@ -173,6 +175,6 @@
 	</joint>
 	<joint name="joint_3" type="revolute">
-        <parent link="arm_link" />
-        <child link="elbow_link" />
+        <parent link="$(arg link_prefix)arm_link" />
+        <child link="$(arg link_prefix)elbow_link" />
         <origin xyz="${distance_arm_elbow_x} ${distance_arm_elbow_y} 0" rpy="0 0 ${-PI/2}" />
 		<limit effort="1" velocity="1.0" lower="${limit_low_elbow_rotation}" upper="${limit_up_elbow_rotation}" />
@@ -180,6 +182,6 @@
 	</joint>
 	<joint name="joint_4" type="revolute">
-        <parent link="elbow_link" />
-        <child link="forearm_link" />
+        <parent link="$(arg link_prefix)elbow_link" />
+        <child link="$(arg link_prefix)forearm_link" />
         <origin xyz="${distance_elbow_forearm_x} ${distance_elbow_forearm_y} 0" rpy="0 ${PI/2} 0" />
 		<limit effort="1" velocity="1.0" lower="${limit_low_forearm_rotation}" upper="${limit_up_forearm_rotation}" />
@@ -187,6 +189,6 @@
 	</joint>
 	<joint name="joint_5" type="revolute">
-        <parent link="forearm_link" />
-        <child link="wrist_link" />
+        <parent link="$(arg link_prefix)forearm_link" />
+        <child link="$(arg link_prefix)wrist_link" />
 		<origin xyz="0 0 ${distance_forearm_wrist_z}" rpy="0 ${-PI/2} 0" />
 		<limit effort="1" velocity="1.0" lower="${limit_low_wrist_rotation}" upper="${limit_up_wrist_rotation}" />
@@ -194,6 +196,6 @@
 	</joint>
 	<joint name="joint_6" type="revolute">
-        <parent link="wrist_link" />
-        <child link="hand_link" />
+        <parent link="$(arg link_prefix)wrist_link" />
+        <child link="$(arg link_prefix)hand_link" />
         <origin xyz="${distance_wrist_hand_x} ${distance_wrist_hand_y} 0" rpy="0 ${PI/2} 0" />
 		<limit effort="1" velocity="1.0" lower="${limit_low_hand_rotation}" upper="${limit_up_hand_rotation}" />
@@ -201,16 +203,16 @@
 	</joint>
 	<joint name="hand_tool_joint" type="fixed">
-        <parent link="hand_link" />
-        <child link="tool_link" />
+        <parent link="$(arg link_prefix)hand_link" />
+        <child link="$(arg link_prefix)tool_link" />
         <origin xyz="0 0 ${distance_hand_tool}" rpy="${-PI/2} ${-PI/2} 0" />
     </joint>
 	<joint name="hand_spoon_joint" type="fixed">
-        <parent link="hand_link" />
-        <child link="spoon_link" />
+        <parent link="$(arg link_prefix)hand_link" />
+        <child link="$(arg link_prefix)spoon_link" />
         <origin xyz="${spoon_offset_left} ${spoon_offset_up} ${spoon_offset_forward}" rpy="0 0 0" />
 	</joint>
     <joint name="kinect_camera_joint" type="fixed">
-        <parent link="base_link" />
-        <child link="camera_rgb_optical_frame" />
+        <parent link="$(arg link_prefix)base_link" />
+        <child link="$(arg link_prefix)camera_rgb_optical_frame" />
         <origin xyz="0 -0.2 0" rpy="0 0 0" />
 	</joint>

File: niryo_one_moveit_config/config/niryo_one.srdf.xacro (robot description, xacro)
@@ -19,5 +19,7 @@
     A URDF file must exist for this robot as well, where the joints and the links that are referenced are defined
 -->
-<robot name="niryo_one">
+<robot xmlns:xacro="http://www.ros.org/wiki/xacro" name="niryo_one">
+    <!-- Add an xacro arg to simulate tf_prefix -->
+    <xacro:arg name="link_prefix" default=""/>
     <!--GROUPS: Representation of a set of joints and links. This can be useful for specifying DOF to plan for, defining arms, end effectors, etc-->
     <!--LINKS: When a link is specified, the parent joint of that link (if it exists) is automatically included-->
@@ -26,8 +28,8 @@
     <!--SUBGROUPS: Groups can also be formed by referencing to already defined group names-->
     <group name="arm">
-        <chain base_link="base_link" tip_link="tool_link" />
+        <chain base_link="$(arg link_prefix)base_link" tip_link="$(arg link_prefix)tool_link" />
     </group>
         <group name="tool">
-        <link name="tool_link" />
+        <link name="$(arg link_prefix)tool_link" />
     </group>
     <!--GROUP STATES: Purpose: Define a named state for a particular group, in terms of joint values. This is useful to define states like 'folded arms'-->
@@ -57,26 +59,26 @@
     </group_state>
     <!--END EFFECTOR: Purpose: Represent information about an end effector.-->
-    <end_effector name="tool_eef" parent_link="tool_link" group="tool" />
+    <end_effector name="tool_eef" parent_link="$(arg link_prefix)tool_link" group="tool" />
     <!--VIRTUAL JOINT: Purpose: this element defines a virtual joint between a robot link and an external frame of reference (considered fixed with respect to the robot)-->
-    <virtual_joint name="fixed_base" type="fixed" parent_frame="world" child_link="ground_link" />
+    <virtual_joint name="fixed_base" type="fixed" parent_frame="world" child_link="$(arg link_prefix)ground_link" />
     <!--DISABLE COLLISIONS: By default it is assumed that any link of the robot could potentially come into collision with any other link in the robot. This tag disables collision checking between a specified pair of links. -->
-    <disable_collisions link1="arm_link" link2="base_link" reason="Never" />
-    <disable_collisions link1="arm_link" link2="elbow_link" reason="Adjacent" />
-    <disable_collisions link1="arm_link" link2="hand_link" reason="Never" />
-    <disable_collisions link1="arm_link" link2="shoulder_link" reason="Adjacent" />
-    <disable_collisions link1="arm_link" link2="wrist_link" reason="Never" />
-    <disable_collisions link1="arm_link" link2="forearm_link" reason="Never" />
-    <disable_collisions link1="base_link" link2="elbow_link" reason="Never" />
-    <disable_collisions link1="base_link" link2="shoulder_link" reason="Adjacent" />
-    <disable_collisions link1="elbow_link" link2="forearm_link" reason="Adjacent" />
-    <disable_collisions link1="elbow_link" link2="tool_link" reason="Never" />
-    <disable_collisions link1="elbow_link" link2="hand_link" reason="Never" />
-    <disable_collisions link1="elbow_link" link2="shoulder_link" reason="Never" />
-    <disable_collisions link1="elbow_link" link2="wrist_link" reason="Never" />
-    <disable_collisions link1="forearm_link" link2="tool_link" reason="Never" />
-    <disable_collisions link1="forearm_link" link2="hand_link" reason="Never" />
-    <disable_collisions link1="forearm_link" link2="wrist_link" reason="Adjacent" />
-    <disable_collisions link1="tool_link" link2="hand_link" reason="Adjacent" />
-    <disable_collisions link1="tool_link" link2="wrist_link" reason="Default" />
-    <disable_collisions link1="hand_link" link2="wrist_link" reason="Adjacent" />
+    <disable_collisions link1="$(arg link_prefix)arm_link" link2="$(arg link_prefix)base_link" reason="Never" />
+    <disable_collisions link1="$(arg link_prefix)arm_link" link2="$(arg link_prefix)elbow_link" reason="Adjacent" />
+    <disable_collisions link1="$(arg link_prefix)arm_link" link2="$(arg link_prefix)hand_link" reason="Never" />
+    <disable_collisions link1="$(arg link_prefix)arm_link" link2="$(arg link_prefix)shoulder_link" reason="Adjacent" />
+    <disable_collisions link1="$(arg link_prefix)arm_link" link2="$(arg link_prefix)wrist_link" reason="Never" />
+    <disable_collisions link1="$(arg link_prefix)arm_link" link2="$(arg link_prefix)forearm_link" reason="Never" />
+    <disable_collisions link1="$(arg link_prefix)base_link" link2="$(arg link_prefix)elbow_link" reason="Never" />
+    <disable_collisions link1="$(arg link_prefix)base_link" link2="$(arg link_prefix)shoulder_link" reason="Adjacent" />
+    <disable_collisions link1="$(arg link_prefix)elbow_link" link2="$(arg link_prefix)forearm_link" reason="Adjacent" />
+    <disable_collisions link1="$(arg link_prefix)elbow_link" link2="$(arg link_prefix)tool_link" reason="Never" />
+    <disable_collisions link1="$(arg link_prefix)elbow_link" link2="$(arg link_prefix)hand_link" reason="Never" />
+    <disable_collisions link1="$(arg link_prefix)elbow_link" link2="$(arg link_prefix)shoulder_link" reason="Never" />
+    <disable_collisions link1="$(arg link_prefix)elbow_link" link2="$(arg link_prefix)wrist_link" reason="Never" />
+    <disable_collisions link1="$(arg link_prefix)forearm_link" link2="$(arg link_prefix)tool_link" reason="Never" />
+    <disable_collisions link1="$(arg link_prefix)forearm_link" link2="$(arg link_prefix)hand_link" reason="Never" />
+    <disable_collisions link1="$(arg link_prefix)forearm_link" link2="$(arg link_prefix)wrist_link" reason="Adjacent" />
+    <disable_collisions link1="$(arg link_prefix)tool_link" link2="$(arg link_prefix)hand_link" reason="Adjacent" />
+    <disable_collisions link1="$(arg link_prefix)tool_link" link2="$(arg link_prefix)wrist_link" reason="Default" />
+    <disable_collisions link1="$(arg link_prefix)hand_link" link2="$(arg link_prefix)wrist_link" reason="Adjacent" />
 </robot>

Commit message: shorten fork, set to version one

File: niryo_one_description/urdf/v2/niryo_one.urdf.xacro (robot description, xacro)
@@ -30,5 +30,6 @@
     <xacro:property name="distance_hand_tool" value="0.0073" />
     <!-- TSR 2018-19-07 Adding info about test spoon-->
-    <xacro:property name="spoon_offset_left" value="0.125" />
+    <!--<xacro:property name="spoon_offset_left" value="0.125" />-->
+    <xacro:property name="spoon_offset_left" value="0.08" />
     <xacro:property name="spoon_offset_up" value="0.0" />
     <xacro:property name="spoon_offset_forward" value="0.031" />
