Commit message: add spoon to v1 urdf

File: niryo_one_description/urdf/v1/niryo_one.urdf.xacro (robot description, xacro)
@@ -24,7 +24,11 @@
     <xacro:property name="distance_elbow_forearm_y" value="0.032" />
     <xacro:property name="distance_forearm_wrist_z" value="0.180" />
-    <xacro:property name="distance_wrist_hand_x" value="0.018" />
-    <xacro:property name="distance_wrist_hand_y" value="0" />
-    <xacro:property name="distance_hand_tool" value="0.00" />
+    <xacro:property name="distance_wrist_hand_x" value="0.0164" />
+    <xacro:property name="distance_wrist_hand_y" value="-0.0055" />
+    <xacro:property name="distance_hand_tool" value="0.0073" />
+    <!-- TSR 2018-19-07 Adding info about test spoon-->
+    <xacro:property name="spoon_offset_left" value="0.125" />
+    <xacro:property name="spoon_offset_up" value="0.0" />
+    <xacro:property name="spoon_offset_forward" value="0.031" />
 	<xacro:property name="PI" value="3.14159265359" />
     <xacro:property name="limit_low_shoulder_rotation" value="-3.05433" />
@@ -162,5 +166,9 @@
         </collision>
 	</link>
-    <link name="tool_link">
+    <link name="$tool_link">
+	</link>
+    <link name="$(arg link_prefix)spoon_link">
+	</link>
+    <link name="$(arg link_prefix)camera_rgb_optical_frame">
 	</link>
 	<!--Joints -->
@@ -216,4 +224,9 @@
         <child link="tool_link" />
         <origin xyz="0 0 ${distance_hand_tool}" rpy="${-PI/2} ${-PI/2} 0" />
+    </joint>
+	<joint name="hand_spoon_joint" type="fixed">
+        <parent link="hand_link" />
+        <child link="spoon_link" />
+        <origin xyz="${spoon_offset_left} ${spoon_offset_up} ${spoon_offset_forward}" rpy="0 0 0" />
 	</joint>
 </robot>

File: niryo_one_description/urdf/v1/without_mesh_niryo_one.urdf.xacro (robot description, xacro)
@@ -27,4 +27,7 @@
     <xacro:property name="distance_wrist_hand_y" value="0" />
     <xacro:property name="distance_hand_tool" value="0.00" />
+    <xacro:property name="spoon_offset_left" value="0.125" />
+    <xacro:property name="spoon_offset_up" value="0.0" />
+    <xacro:property name="spoon_offset_forward" value="0.031" />
 	<xacro:property name="PI" value="3.14159265359" />
 	<xacro:property name="limit_low_shoulder_rotation" value="-3.05433" />
@@ -110,4 +113,9 @@
         <child link="tool_link" />
         <origin xyz="0 0 ${distance_hand_tool}" rpy="${-PI/2} ${-PI/2} 0" />
+    </joint>
+	<joint name="hand_spoon_joint" type="fixed">
+        <parent link="hand_link" />
+        <child link="spoon_link" />
+        <origin xyz="${spoon_offset_left} ${spoon_offset_up} ${spoon_offset_forward}" rpy="0 0 0" />
 	</joint>
 </robot>

Commit message: forgot to add spoon link

File: niryo_one_description/urdf/v1/niryo_one.urdf.xacro (robot description, xacro)
@@ -168,7 +168,5 @@
     <link name="$tool_link">
 	</link>
-    <link name="$(arg link_prefix)spoon_link">
-	</link>
-    <link name="$(arg link_prefix)camera_rgb_optical_frame">
+    <link name="spoon_link">
 	</link>
 	<!--Joints -->

File: niryo_one_description/urdf/v1/without_mesh_niryo_one.urdf.xacro (robot description, xacro)
@@ -61,4 +61,6 @@
     <link name="tool_link">
 	</link>
+    <link name="spoon_link">
+	</link>
 	<!--Joints -->
     <joint name="ground_joint" type="fixed">

Commit message: not sure why these numbers are different from niryo's github, but revert them back to match

File: niryo_one_description/urdf/v1/niryo_one.urdf.xacro (robot description, xacro)
@@ -24,7 +24,7 @@
     <xacro:property name="distance_elbow_forearm_y" value="0.032" />
     <xacro:property name="distance_forearm_wrist_z" value="0.180" />
-    <xacro:property name="distance_wrist_hand_x" value="0.0164" />
-    <xacro:property name="distance_wrist_hand_y" value="-0.0055" />
-    <xacro:property name="distance_hand_tool" value="0.0073" />
+    <xacro:property name="distance_wrist_hand_x" value="0.018" />
+    <xacro:property name="distance_wrist_hand_y" value="0" />
+    <xacro:property name="distance_hand_tool" value="0.00" />
     <!-- TSR 2018-19-07 Adding info about test spoon-->
     <xacro:property name="spoon_offset_left" value="0.125" />

File: niryo_one_description/urdf/v2/niryo_one.urdf.xacro (robot description, xacro)
@@ -23,6 +23,6 @@
     <xacro:property name="distance_arm_elbow_x" value="0.210" />
     <xacro:property name="distance_arm_elbow_y" value="0.0" />
-    <xacro:property name="distance_elbow_forearm_x" value="0.037" />
-    <xacro:property name="distance_elbow_forearm_y" value="0.032" />
+    <xacro:property name="distance_elbow_forearm_x" value="0.0415" />
+    <xacro:property name="distance_elbow_forearm_y" value="0.030" />
     <xacro:property name="distance_forearm_wrist_z" value="0.180" />
     <xacro:property name="distance_wrist_hand_x" value="0.0164" />

Commit message: I'm such a klutz

File: niryo_one_description/urdf/v1/niryo_one.urdf.xacro (robot description, xacro)
@@ -166,5 +166,5 @@
         </collision>
 	</link>
-    <link name="$tool_link">
+    <link name="tool_link">
 	</link>
     <link name="spoon_link">

Commit message: get a floppy robot to appear in gazebo

File: niryo_one_description/urdf/v1/niryo_one.urdf.xacro (robot description, xacro)
@@ -16,4 +16,6 @@
 -->
 <robot xmlns:xacro="http://www.ros.org/wiki/xacro" name="niryo_one">
+  <!-- Import all Gazebo-customization elements, including Gazebo colors -->
+  <xacro:include filename="$(find niryo_one_description)/urdf/v1/niryo_one.gazebo" />
 	<!-- Properties -->
     <xacro:property name="distance_origin_shoulder_z" value="0.103" />
@@ -31,4 +33,8 @@
     <xacro:property name="spoon_offset_up" value="0.0" />
     <xacro:property name="spoon_offset_forward" value="0.031" />
+    <!-- TSR 2018-19-07 Adding info about camera -->
+    <xacro:property name="camera_width" value="0.01" />
+    <xacro:property name="camera_pitch" value="0.3" />
+    <xacro:property name="camera_height" value="0.04" />
 	<xacro:property name="PI" value="3.14159265359" />
     <xacro:property name="limit_low_shoulder_rotation" value="-3.05433" />
@@ -45,4 +51,10 @@
     <xacro:property name="limit_up_hand_rotation" value="2.57" />
 	<!-- Links -->
+  <!-- Used for fixing robot to Gazebo 'base_link' -->
+  <link name="world"/>
+  <joint name="fixed" type="fixed">
+    <parent link="world"/>
+    <child link="ground_link"/>
+  </joint>
     <link name="ground_link"/>
     <link name="base_link">
@@ -62,4 +74,12 @@
             </geometry>
         </collision>
+        <inertial>
+          <origin xyz="0 0 ${distance_origin_shoulder_z/2}" rpy="0 0 0"/>
+          <mass value="0.5"/>
+          <inertia
+            ixx="1.0" ixy="0.0" ixz="0.0"
+            iyy="1.0" iyz="0.0"
+            izz="1.0"/>
+        </inertial>
 	</link>
     <link name="shoulder_link">
@@ -79,4 +99,12 @@
             </geometry>
         </collision>
+        <inertial>
+          <origin xyz="0 0 ${distance_shoulder_arm_z/2}" rpy="0 0 0"/>
+          <mass value="0.5"/>
+          <inertia
+            ixx="1.0" ixy="0.0" ixz="0.0"
+            iyy="1.0" iyz="0.0"
+            izz="1.0"/>
+        </inertial>
 	</link>
     <link name="arm_link">
@@ -96,4 +124,12 @@
             </geometry>
         </collision>
+        <inertial>
+          <origin xyz="${distance_arm_elbow_x/2} ${distance_arm_elbow_y/2} 0" rpy="0 0 0"/>
+          <mass value="0.5"/>
+          <inertia
+            ixx="1.0" ixy="0.0" ixz="0.0"
+            iyy="1.0" iyz="0.0"
+            izz="1.0"/>
+        </inertial>
 	</link>
     <link name="elbow_link">
@@ -114,4 +150,12 @@
             </geometry>
         </collision>
+        <inertial>
+          <origin xyz="${distance_elbow_forearm_x/2} ${distance_elbow_forearm_y/2} 0" rpy="0 0 0"/>
+          <mass value="0.5"/>
+          <inertia
+            ixx="1.0" ixy="0.0" ixz="0.0"
+            iyy="1.0" iyz="0.0"
+            izz="1.0"/>
+        </inertial>
 	</link>
     <link name="forearm_link">
@@ -131,4 +175,12 @@
             </geometry>
         </collision>
+        <inertial>
+          <origin xyz="0 0 ${distance_forearm_wrist_z/2}" rpy="0 0 0"/>
+          <mass value="0.5"/>
+          <inertia
+            ixx="1.0" ixy="0.0" ixz="0.0"
+            iyy="1.0" iyz="0.0"
+            izz="1.0"/>
+        </inertial>
 	</link>
     <link name="wrist_link">
@@ -148,4 +200,12 @@
             </geometry>
         </collision>
+        <inertial>
+          <origin xyz="${distance_wrist_hand_x/2} ${distance_wrist_hand_y/2} 0" rpy="0 0 0"/>
+          <mass value="0.5"/>
+          <inertia
+            ixx="1.0" ixy="0.0" ixz="0.0"
+            iyy="1.0" iyz="0.0"
+            izz="1.0"/>
+        </inertial>
 	</link>
     <link name="hand_link">
@@ -165,9 +225,72 @@
             </geometry>
         </collision>
+        <inertial>
+          <origin xyz="0 0 0" rpy="0 0 0"/>
+          <mass value="0.5"/>
+          <inertia
+            ixx="1.0" ixy="0.0" ixz="0.0"
+            iyy="1.0" iyz="0.0"
+            izz="1.0"/>
+        </inertial>
 	</link>
     <link name="tool_link">
 	</link>
     <link name="spoon_link">
-	</link>
+		<visual>
+			<origin xyz="0 0 0" rpy="0 0 0" />
+			<geometry>
+                <mesh filename="package://niryo_one_description/meshes/v1/stl/spoon.stl" />
+			</geometry>
+			<material name="">
+				<color rgba="0.6 0 0 1" />
+			</material>
+		</visual>
+        <collision>
+			<origin xyz="0 0 0" rpy="0 0 0" />
+            <geometry>
+                <mesh filename="package://niryo_one_description/meshes/v1/stl/spoon.stl" />
+            </geometry>
+        </collision>
+        <inertial>
+          <origin xyz="0 0 0" rpy="0 0 0"/>
+          <mass value="0.5"/>
+          <inertia
+            ixx="1.0" ixy="0.0" ixz="0.0"
+            iyy="1.0" iyz="0.0"
+            izz="1.0"/>
+        </inertial>
+	</link>
+  <!-- Camera -->
+  <link name="camera_link">
+    <collision>
+      <origin xyz="0 0 0" rpy="0 0 0"/>
+      <geometry>
+	<box size="${camera_width} ${camera_width} ${camera_width}"/>
+      </geometry>
+    </collision>
+    <visual>
+      <origin xyz="0 0 0" rpy="0 0 0"/>
+      <geometry>
+	<box size="${camera_width} ${camera_width} ${camera_width}"/>
+      </geometry>
+      <material name="red"/>
+    </visual>
+    <inertial>
+      <mass value="1e-5" />
+      <origin xyz="0 0 0" rpy="0 0 0"/>
+      <inertia ixx="1e-6" ixy="0" ixz="0" iyy="1e-6" iyz="0" izz="1e-6" />
+    </inertial>
+  </link>
+  <!-- generate an optical frame http://www.ros.org/reps/rep-0103.html#suffix-frames
+      so that ros and opencv can operate on the camera frame correctly -->
+  <joint name="camera_optical_joint" type="fixed">
+    <!-- these values have to be these values otherwise the gazebo camera image
+        won't be aligned properly with the frame it is supposedly originating from -->
+    <origin xyz="0 0 0" rpy="${-pi/2} 0 ${-pi/2}"/>
+    <parent link="camera_link"/>
+    <child link="camera_link_optical"/>
+  </joint>
+  <link name="camera_link_optical">
+  </link>
 	<!--Joints -->
     <joint name="ground_joint" type="fixed">
@@ -222,5 +345,10 @@
         <child link="tool_link" />
         <origin xyz="0 0 ${distance_hand_tool}" rpy="${-PI/2} ${-PI/2} 0" />
-    </joint>
+        </joint>
+	<joint name="camera_link_joint" type="fixed">
+        <parent link="hand_link" />
+        <child link="camera_link" />
+        <origin xyz="0.01 ${camera_height} ${spoon_offset_forward}" rpy="${-PI/2} 0 ${-camera_pitch}" />
+        </joint>
 	<joint name="hand_spoon_joint" type="fixed">
         <parent link="hand_link" />

Commit message: get gazebo to work

File: niryo_one_description/urdf/v1/niryo_one.urdf.xacro (robot description, xacro)
@@ -76,9 +76,9 @@
         <inertial>
           <origin xyz="0 0 ${distance_origin_shoulder_z/2}" rpy="0 0 0"/>
-          <mass value="0.5"/>
-          <inertia
-            ixx="1.0" ixy="0.0" ixz="0.0"
-            iyy="1.0" iyz="0.0"
-            izz="1.0"/>
+          <mass value="0.05"/>
+          <inertia
+            ixx="1e-3" ixy="0.0" ixz="0.0"
+            iyy="1e-3" iyz="0.0"
+            izz="1e-3"/>
         </inertial>
 	</link>
@@ -101,9 +101,9 @@
         <inertial>
           <origin xyz="0 0 ${distance_shoulder_arm_z/2}" rpy="0 0 0"/>
-          <mass value="0.5"/>
-          <inertia
-            ixx="1.0" ixy="0.0" ixz="0.0"
-            iyy="1.0" iyz="0.0"
-            izz="1.0"/>
+          <mass value="0.05"/>
+          <inertia
+            ixx="1e-3" ixy="0.0" ixz="0.0"
+            iyy="1e-3" iyz="0.0"
+            izz="1e-3"/>
         </inertial>
 	</link>
@@ -126,9 +126,9 @@
         <inertial>
           <origin xyz="${distance_arm_elbow_x/2} ${distance_arm_elbow_y/2} 0" rpy="0 0 0"/>
-          <mass value="0.5"/>
-          <inertia
-            ixx="1.0" ixy="0.0" ixz="0.0"
-            iyy="1.0" iyz="0.0"
-            izz="1.0"/>
+          <mass value="0.05"/>
+          <inertia
+            ixx="1e-3" ixy="0.0" ixz="0.0"
+            iyy="1e-3" iyz="0.0"
+            izz="1e-3"/>
         </inertial>
 	</link>
@@ -152,9 +152,9 @@
         <inertial>
           <origin xyz="${distance_elbow_forearm_x/2} ${distance_elbow_forearm_y/2} 0" rpy="0 0 0"/>
-          <mass value="0.5"/>
-          <inertia
-            ixx="1.0" ixy="0.0" ixz="0.0"
-            iyy="1.0" iyz="0.0"
-            izz="1.0"/>
+          <mass value="0.05"/>
+          <inertia
+            ixx="1e-3" ixy="0.0" ixz="0.0"
+            iyy="1e-3" iyz="0.0"
+            izz="1e-3"/>
         </inertial>
 	</link>
@@ -177,9 +177,9 @@
         <inertial>
           <origin xyz="0 0 ${distance_forearm_wrist_z/2}" rpy="0 0 0"/>
-          <mass value="0.5"/>
-          <inertia
-            ixx="1.0" ixy="0.0" ixz="0.0"
-            iyy="1.0" iyz="0.0"
-            izz="1.0"/>
+          <mass value="0.05"/>
+          <inertia
+            ixx="1e-3" ixy="0.0" ixz="0.0"
+            iyy="1e-3" iyz="0.0"
+            izz="1e-3"/>
         </inertial>
 	</link>
@@ -202,9 +202,9 @@
         <inertial>
           <origin xyz="${distance_wrist_hand_x/2} ${distance_wrist_hand_y/2} 0" rpy="0 0 0"/>
-          <mass value="0.5"/>
-          <inertia
-            ixx="1.0" ixy="0.0" ixz="0.0"
-            iyy="1.0" iyz="0.0"
-            izz="1.0"/>
+          <mass value="0.05"/>
+          <inertia
+            ixx="1e-3" ixy="0.0" ixz="0.0"
+            iyy="1e-3" iyz="0.0"
+            izz="1e-3"/>
         </inertial>
 	</link>
@@ -227,9 +227,9 @@
         <inertial>
           <origin xyz="0 0 0" rpy="0 0 0"/>
-          <mass value="0.5"/>
-          <inertia
-            ixx="1.0" ixy="0.0" ixz="0.0"
-            iyy="1.0" iyz="0.0"
-            izz="1.0"/>
+          <mass value="0.05"/>
+          <inertia
+            ixx="1e-3" ixy="0.0" ixz="0.0"
+            iyy="1e-3" iyz="0.0"
+            izz="1e-3"/>
         </inertial>
 	</link>
@@ -253,10 +253,10 @@
         </collision>
         <inertial>
-          <origin xyz="0 0 0" rpy="0 0 0"/>
-          <mass value="0.5"/>
-          <inertia
-            ixx="1.0" ixy="0.0" ixz="0.0"
-            iyy="1.0" iyz="0.0"
-            izz="1.0"/>
+          <origin xyz="${-spoon_offset_left} 0 0" rpy="0 0 0"/>
+          <mass value="0.05"/>
+          <inertia
+            ixx="1e-3" ixy="0.0" ixz="0.0"
+            iyy="1e-3" iyz="0.0"
+            izz="1e-3"/>
         </inertial>
 	</link>
@@ -356,3 +356,64 @@
         <origin xyz="${spoon_offset_left} ${spoon_offset_up} ${spoon_offset_forward}" rpy="0 0 0" />
 	</joint>
+<!-- Actuators -->
+<transmission name="transmission_1">
+  <type>transmission_interface/SimpleTransmission</type>
+  <joint name="joint_1">
+    <hardwareInterface>hardware_interface/EffortJointInterface</hardwareInterface>
+  </joint>
+  <actuator name="stepper_motor_1">
+    <hardwareInterface>hardware_interface/EffortJointInterface</hardwareInterface>
+    <mechanicalReduction>50</mechanicalReduction>
+  </actuator>
+</transmission>
+<transmission name="transmission_2">
+  <type>transmission_interface/SimpleTransmission</type>
+  <joint name="joint_2">
+    <hardwareInterface>hardware_interface/EffortJointInterface</hardwareInterface>
+  </joint>
+  <actuator name="stepper_motor_2">
+    <hardwareInterface>hardware_interface/EffortJointInterface</hardwareInterface>
+    <mechanicalReduction>50</mechanicalReduction>
+  </actuator>
+</transmission>
+<transmission name="transmission_3">
+  <type>transmission_interface/SimpleTransmission</type>
+  <joint name="joint_3">
+    <hardwareInterface>hardware_interface/EffortJointInterface</hardwareInterface>
+  </joint>
+  <actuator name="stepper_motor_3">
+    <hardwareInterface>hardware_interface/EffortJointInterface</hardwareInterface>
+    <mechanicalReduction>50</mechanicalReduction>
+  </actuator>
+</transmission>
+<transmission name="transmission_4">
+  <type>transmission_interface/SimpleTransmission</type>
+  <joint name="joint_4">
+    <hardwareInterface>hardware_interface/EffortJointInterface</hardwareInterface>
+  </joint>
+  <actuator name="stepper_motor_4">
+    <hardwareInterface>hardware_interface/EffortJointInterface</hardwareInterface>
+    <mechanicalReduction>50</mechanicalReduction>
+  </actuator>
+</transmission>
+<transmission name="transmission_5">
+  <type>transmission_interface/SimpleTransmission</type>
+  <joint name="joint_5">
+    <hardwareInterface>hardware_interface/EffortJointInterface</hardwareInterface>
+  </joint>
+  <actuator name="stepper_motor_5">
+    <hardwareInterface>hardware_interface/EffortJointInterface</hardwareInterface>
+    <mechanicalReduction>50</mechanicalReduction>
+  </actuator>
+</transmission>
+<transmission name="transmission_6">
+  <type>transmission_interface/SimpleTransmission</type>
+  <joint name="joint_6">
+    <hardwareInterface>hardware_interface/EffortJointInterface</hardwareInterface>
+  </joint>
+  <actuator name="stepper_motor_6">
+    <hardwareInterface>hardware_interface/EffortJointInterface</hardwareInterface>
+    <mechanicalReduction>50</mechanicalReduction>
+  </actuator>
+</transmission>
 </robot>

Commit message: put niryo on table

File: niryo_one_description/urdf/v1/niryo_one.urdf.xacro (robot description, xacro)
@@ -56,4 +56,5 @@
     <parent link="world"/>
     <child link="ground_link"/>
+    <origin xyz="0 0 1.02" rpy="0 0 0" />
   </joint>
     <link name="ground_link"/>
